Commit message: Gazebo world ready: robot spawned, gravity disabled, meshes fixed

File: src/MG400_ROS2/mg400_description/urdf/mg400.urdf.xacro (robot description, xacro)
@@ -1,26 +1,43 @@
 <?xml version="1.0" encoding="utf-8"?>
-<robot
-        xmlns:xacro="http://ros.org/wiki/xacro"
-        name="mg400">
+<robot xmlns:xacro="http://ros.org/wiki/xacro" name="mg400">
     <xacro:include filename="$(find mg400_description)/urdf/mg400.xacro" />
-    <!-- arguments -->
-    <xacro:arg
-            name="prefix"
-            default="" />
-    <xacro:arg
-            name="use_arm"
-            default="True" />
-    <xacro:arg
-            name="workspace_visible"
-            default="false" />
-    <!-- links -->
-    <link name="$(arg prefix)arm_frame_link_offset" />
+    <xacro:arg name="prefix" default="" />
+    <xacro:arg name="use_arm" default="True" />
+    <xacro:arg name="workspace_visible" default="false" />
+    <link name="world" />
+    <joint name="world_fixed_joint" type="fixed">
+        <parent link="world" />
+        <child link="$(arg prefix)arm_frame_link_offset" />
+        <origin xyz="0 0 0" rpy="0 0 0" />
+    </joint>
+    <link name="$(arg prefix)arm_frame_link_offset">
+        <inertial>
+            <mass value="10.0"/>
+            <origin xyz="0 0 0" rpy="0 0 0"/>
+            <inertia ixx="0.1" ixy="0" ixz="0" iyy="0.1" iyz="0" izz="0.1"/>
+        </inertial>
+        <collision>
+            <origin xyz="0 0 0" rpy="0 0 0"/>
+            <geometry><box size="0.1 0.1 0.1"/></geometry>
+        </collision>
+    </link>
     <xacro:mg400
             parent="$(arg prefix)arm_frame_link_offset"
             prefix="$(arg prefix)"
             workspace_visible="$(arg workspace_visible)">
-        <origin
-                xyz="0 0 0"
-                rpy="0 0 0" />
+        <origin xyz="0 0 0" rpy="0 0 0" />
     </xacro:mg400>
+    <gazebo>
+        <static>true</static>
+    </gazebo>
+    <gazebo reference="mg400_base_link"><gravity>0</gravity></gazebo>
+    <gazebo reference="mg400_link1"><gravity>0</gravity></gazebo>
+    <gazebo reference="mg400_link2_1"><gravity>0</gravity></gazebo>
+    <gazebo reference="mg400_link2_2"><gravity>0</gravity></gazebo>
+    <gazebo reference="mg400_link3_1"><gravity>0</gravity></gazebo>
+    <gazebo reference="mg400_link3_2"><gravity>0</gravity></gazebo>
+    <gazebo reference="mg400_link4_1"><gravity>0</gravity></gazebo>
+    <gazebo reference="mg400_link4_2"><gravity>0</gravity></gazebo>
+    <gazebo reference="mg400_link4_3"><gravity>0</gravity></gazebo>
+    <gazebo reference="mg400_link5"><gravity>0</gravity></gazebo>
 </robot>

Commit message: WIP: Patched Gazebo trajectory plugin (bypassed frame_id bug). Fixed dobot_logic setup & bridge. RViz logic 100% ready.

File: src/MG400_ROS2/mg400_description/urdf/mg400.urdf.xacro (robot description, xacro)
@@ -28,6 +28,6 @@
         <origin xyz="0 0 0" rpy="0 0 0" />
     </xacro:mg400>
-    <gazebo>
-        <static>true</static>
+    <gazebo reference="arm_frame_link_offset">
+        <gravity>0</gravity>
     </gazebo>
     <gazebo reference="mg400_base_link"><gravity>0</gravity></gazebo>
@@ -41,3 +41,14 @@
     <gazebo reference="mg400_link4_3"><gravity>0</gravity></gazebo>
     <gazebo reference="mg400_link5"><gravity>0</gravity></gazebo>
+    <gazebo reference="mg400_end_effector_flange"><gravity>0</gravity></gazebo>
+   <gazebo>
+    <static>true</static>
+   </gazebo>
+   <gazebo>
+       <plugin name="gazebo_ros_joint_pose_trajectory" filename="libgazebo_ros_joint_pose_trajectory.so">
+           <ros>
+           </ros>
+           <update_rate>30</update_rate>
+       </plugin>
+   </gazebo>
 </robot>

File: src/MG400_ROS2/mg400_description/urdf/mg400.xacro (robot description, xacro)
@@ -6,46 +6,18 @@
       ns="const" />
   <!-- Base path for meshes -->
-  <xacro:property
-      name="BASE_PATH"
-      value="mg400_description/meshes" />
-  <xacro:property
-      name="MESH_BASE_LINK"
-      value="${BASE_PATH}/base_link.dae" />
-  <xacro:property
-      name="MESH_LINK_1"
-      value="${BASE_PATH}/link1.dae" />
-  <xacro:property
-      name="MESH_LINK_2_1"
-      value="${BASE_PATH}/link2_1.dae" />
-  <xacro:property
-      name="MESH_LINK_2_2"
-      value="${BASE_PATH}/link2_2.dae" />
-  <xacro:property
-      name="MESH_LINK_3_1"
-      value="${BASE_PATH}/link3_1.dae" />
-  <xacro:property
-      name="MESH_LINK_3_2"
-      value="${BASE_PATH}/link3_2.dae" />
-  <xacro:property
-      name="MESH_LINK_4_1"
-      value="${BASE_PATH}/link4_1.dae" />
-  <xacro:property
-      name="MESH_LINK_4_2"
-      value="${BASE_PATH}/link4_2.dae" />
-  <xacro:property
-      name="MESH_LINK_4_3"
-      value="${BASE_PATH}/link4_3.dae" />
-  <xacro:property
-      name="MESH_LINK_5"
-      value="${BASE_PATH}/link5.dae" />
-  <xacro:property
-      name="MESH_FLANGE"
-      value="${BASE_PATH}/flange.dae" />
-  <xacro:property
-      name="MESH_WORKSPACE"
-      value="${BASE_PATH}/workspace.dae" />
-  <xacro:macro
-      name="mg400"
-      params="prefix parent *origin workspace_visible">
+  <xacro:property name="BASE_PATH" value="mg400_description/meshes" />
+  <xacro:property name="MESH_BASE_LINK" value="${BASE_PATH}/base_link.dae" />
+  <xacro:property name="MESH_LINK_1" value="${BASE_PATH}/link1.dae" />
+  <xacro:property name="MESH_LINK_2_1" value="${BASE_PATH}/link2_1.dae" />
+  <xacro:property name="MESH_LINK_2_2" value="${BASE_PATH}/link2_2.dae" />
+  <xacro:property name="MESH_LINK_3_1" value="${BASE_PATH}/link3_1.dae" />
+  <xacro:property name="MESH_LINK_3_2" value="${BASE_PATH}/link3_2.dae" />
+  <xacro:property name="MESH_LINK_4_1" value="${BASE_PATH}/link4_1.dae" />
+  <xacro:property name="MESH_LINK_4_2" value="${BASE_PATH}/link4_2.dae" />
+  <xacro:property name="MESH_LINK_4_3" value="${BASE_PATH}/link4_3.dae" />
+  <xacro:property name="MESH_LINK_5" value="${BASE_PATH}/link5.dae" />
+  <xacro:property name="MESH_FLANGE" value="${BASE_PATH}/flange.dae" />
+  <xacro:property name="MESH_WORKSPACE" value="${BASE_PATH}/workspace.dae" />
+  <xacro:macro name="mg400" params="prefix parent *origin workspace_visible">
     <material name="${prefix}mg400_workspace_material">
       <color rgba="0.2 0.0 0.0 0.5" />
@@ -54,31 +26,16 @@
     <link name="${prefix}mg400_base_link">
       <inertial>
-        <origin
-            xyz="0.000600637001378879 -2.53487071137343E-07 0.0560927888040551"
-            rpy="0 0 0" />
+        <origin xyz="0.000600637001378879 -2.53487071137343E-07 0.0560927888040551" rpy="0 0 0" />
         <mass value="3.62164811695094" />
-        <inertia
-            ixx="0.0126582175296405"
-            ixy="6.66832041405407E-08"
-            ixz="-3.52548281362717E-06"
-            iyy="0.0145891535260188"
-            iyz="5.15901657460475E-08"
-            izz="0.0195045116656827" />
-      </inertial>
-      <visual>
-        <origin
-            xyz="0 0 0"
-            rpy="0 0 0" />
-        <geometry>
-          <mesh filename="package://${MESH_BASE_LINK}" />
-        </geometry>
-      </visual>
-      <collision>
-        <origin
-            xyz="0 0 0"
-            rpy="0 0 0" />
-        <geometry>
-          <mesh filename="package://${MESH_BASE_LINK}" />
-        </geometry>
+        <inertia ixx="0.0126582175296405" ixy="6.66832041405407E-08" ixz="-3.52548281362717E-06"
+                 iyy="0.0145891535260188" iyz="5.15901657460475E-08" izz="0.0195045116656827" />
+      </inertial>
+      <visual>
+        <origin xyz="0 0 0" rpy="0 0 0" />
+        <geometry><mesh filename="package://${MESH_BASE_LINK}" /></geometry>
+      </visual>
+      <collision>
+        <origin xyz="0 0 0" rpy="0 0 0" />
+        <geometry><mesh filename="package://${MESH_BASE_LINK}" /></geometry>
       </collision>
     </link>
@@ -86,310 +43,160 @@
     <link name="${prefix}mg400_link1">
       <inertial>
-        <origin
-            xyz="-0.0046209286967387 -6.88107982318643E-05 0.0709919358465827"
-            rpy="0 0 0" />
+        <origin xyz="-0.0046209286967387 -6.88107982318643E-05 0.0709919358465827" rpy="0 0 0" />
         <mass value="1.77056222753813" />
-        <inertia
-            ixx="0.00605885293080088"
-            ixy="0.000156081820035162"
-            ixz="-0.00021785654850453"
-            iyy="0.00579381982249127"
-            iyz="6.20876898015621E-05"
-            izz="0.00741058257251941" />
-      </inertial>
-      <visual>
-        <origin
-            xyz="0 0 0"
-            rpy="0 0 0" />
-        <geometry>
-          <mesh filename="package://${MESH_LINK_1}" />
-        </geometry>
-      </visual>
-      <collision>
-        <origin
-            xyz="0 0 0"
-            rpy="0 0 0" />
-        <geometry>
-          <mesh filename="package://${MESH_LINK_1}" />
-        </geometry>
+        <inertia ixx="0.00605885293080088" ixy="0.000156081820035162" ixz="-0.00021785654850453"
+                 iyy="0.00579381982249127" iyz="6.20876898015621E-05" izz="0.00741058257251941" />
+      </inertial>
+      <visual>
+        <origin xyz="0 0 0" rpy="0 0 0" />
+        <geometry><mesh filename="package://${MESH_LINK_1}" /></geometry>
+      </visual>
+      <collision>
+        <origin xyz="0 0 0" rpy="0 0 0" />
+        <geometry><mesh filename="package://${MESH_LINK_1}" /></geometry>
       </collision>
     </link>
     <link name="${prefix}mg400_link2_1">
       <inertial>
-        <origin
-            xyz="-0.00321788524756698 0.0352926570826593 0.0596131328734945"
-            rpy="0 0 0" />
+        <origin xyz="-0.00321788524756698 0.0352926570826593 0.0596131328734945" rpy="0 0 0" />
         <mass value="0.0866115884541459" />
-        <inertia
-            ixx="0.000338551627157209"
-            ixy="-2.78858228577314E-09"
-            ixz="1.05212346076681E-05"
-            iyy="0.000307789653713489"
-            iyz="-1.36109590152488E-06"
-            izz="3.89949940178023E-05" />
-      </inertial>
-      <visual>
-        <origin
-            xyz="0 0 0"
-            rpy="0 0 0" />
-        <geometry>
-          <mesh filename="package://${MESH_LINK_2_1}" />
-        </geometry>
-      </visual>
-      <collision>
-        <origin
-            xyz="0 0 0"
-            rpy="0 0 0" />
-        <geometry>
-          <mesh filename="package://${MESH_LINK_2_1}" />
-        </geometry>
+        <inertia ixx="0.000338551627157209" ixy="-2.78858228577314E-09" ixz="1.05212346076681E-05"
+                 iyy="0.000307789653713489" iyz="-1.36109590152488E-06" izz="3.89949940178023E-05" />
+      </inertial>
+      <visual>
+        <origin xyz="0 0 0" rpy="0 0 0" />
+        <geometry><mesh filename="package://${MESH_LINK_2_1}" /></geometry>
+      </visual>
+      <collision>
+        <origin xyz="0 0 0" rpy="0 0 0" />
+        <geometry><mesh filename="package://${MESH_LINK_2_1}" /></geometry>
       </collision>
     </link>
     <link name="${prefix}mg400_link2_2">
       <inertial>
-        <origin
-            xyz="-0.0201111131723385 0.0304999635268521 0.073632809340276"
-            rpy="0 0 0" />
+        <origin xyz="-0.0201111131723385 0.0304999635268521 0.073632809340276" rpy="0 0 0" />
         <mass value="0.0662546292985346" />
-        <inertia
-            ixx="0.000218973873589181"
-            ixy="3.0147933007673E-10"
-            ixz="2.51402553227571E-06"
-            iyy="0.000200510070261609"
-            iyz="-1.41837669904595E-09"
-            izz="3.74316777806776E-05" />
-      </inertial>
-      <visual>
-        <origin
-            xyz="0 0 0"
-            rpy="0 0 0" />
-        <geometry>
-          <mesh filename="package://${MESH_LINK_2_2}" />
-        </geometry>
-      </visual>
-      <collision>
-        <origin
-            xyz="0 0 0"
-            rpy="0 0 0" />
-        <geometry>
-          <mesh filename="package://${MESH_LINK_2_2}" />
-        </geometry>
+        <inertia ixx="0.000218973873589181" ixy="3.0147933007673E-10" ixz="2.51402553227571E-06"
+                 iyy="0.000200510070261609" iyz="-1.41837669904595E-09" izz="3.74316777806776E-05" />
+      </inertial>
+      <visual>
+        <origin xyz="0 0 0" rpy="0 0 0" />
+        <geometry><mesh filename="package://${MESH_LINK_2_2}" /></geometry>
+      </visual>
+      <collision>
+        <origin xyz="0 0 0" rpy="0 0 0" />
+        <geometry><mesh filename="package://${MESH_LINK_2_2}" /></geometry>
       </collision>
     </link>
     <link name="${prefix}mg400_link3_1">
       <inertial>
-        <origin
-            xyz="0.0821679417596488 0.000113044685842874 -0.00333758753063973"
-            rpy="0 0 0" />
+        <origin xyz="0.0821679417596488 0.000113044685842874 -0.00333758753063973" rpy="0 0 0" />
         <mass value="0.0375214831045061" />
-        <inertia
-            ixx="2.54761091812684E-06"
-            ixy="3.73102654491378E-07"
-            ixz="-2.02625705871199E-06"
-            iyy="0.000164234314177935"
-            iyz="-1.44731096825347E-08"
-            izz="0.000164331500854172" />
-      </inertial>
-      <visual>
-        <origin
-            xyz="0 0 0"
-            rpy="0 0 0" />
-        <geometry>
-          <mesh filename="package://${MESH_LINK_3_1}" />
-        </geometry>
-      </visual>
-      <collision>
-        <origin
-            xyz="0 0 0"
-            rpy="0 0 0" />
-        <geometry>
-          <mesh filename="package://${MESH_LINK_3_1}" />
-        </geometry>
+        <inertia ixx="2.54761091812684E-06" ixy="3.73102654491378E-07" ixz="-2.02625705871199E-06"
+                 iyy="0.000164234314177935" iyz="-1.44731096825347E-08" izz="0.000164331500854172" />
+      </inertial>
+      <visual>
+        <origin xyz="0 0 0" rpy="0 0 0" />
+        <geometry><mesh filename="package://${MESH_LINK_3_1}" /></geometry>
+      </visual>
+      <collision>
+        <origin xyz="0 0 0" rpy="0 0 0" />
+        <geometry><mesh filename="package://${MESH_LINK_3_1}" /></geometry>
       </collision>
     </link>
     <link name="${prefix}mg400_link3_2">
       <inertial>
-        <origin
-            xyz="0.0338566736074436 0.0240208873857428 0.00452229895926692"
-            rpy="0 0 0" />
+        <origin xyz="0.0338566736074436 0.0240208873857428 0.00452229895926692" rpy="0 0 0" />
         <mass value="0.0366692789294813" />
-        <inertia
-            ixx="7.24011830695354E-06"
-            ixy="7.93542746250724E-10"
-            ixz="-1.69163254472566E-06"
-            iyy="2.34967008246727E-05"
-            iyz="4.55507111386579E-10"
-            izz="1.66831643179488E-05" />
-      </inertial>
-      <visual>
-        <origin
-            xyz="0 0 0"
-            rpy="0 0 0" />
-        <geometry>
-          <mesh filename="package://${MESH_LINK_3_2}" />
-        </geometry>
-      </visual>
-      <collision>
-        <origin
-            xyz="0 0 0"
-            rpy="0 0 0" />
-        <geometry>
-          <mesh filename="package://${MESH_LINK_3_2}" />
-        </geometry>
+        <inertia ixx="7.24011830695354E-06" ixy="7.93542746250724E-10" ixz="-1.69163254472566E-06"
+                 iyy="2.34967008246727E-05" iyz="4.55507111386579E-10" izz="1.66831643179488E-05" />
+      </inertial>
+      <visual>
+        <origin xyz="0 0 0" rpy="0 0 0" />
+        <geometry><mesh filename="package://${MESH_LINK_3_2}" /></geometry>
+      </visual>
+      <collision>
+        <origin xyz="0 0 0" rpy="0 0 0" />
+        <geometry><mesh filename="package://${MESH_LINK_3_2}" /></geometry>
       </collision>
     </link>
     <link name="${prefix}mg400_link4_1">
       <inertial>
-        <origin
-            xyz="0.0387878182928232 0.0170848333998282 -0.0024610990490942"
-            rpy="0 0 0" />
+        <origin xyz="0.0387878182928232 0.0170848333998282 -0.0024610990490942" rpy="0 0 0" />
         <mass value="0.0628979533925801" />
-        <inertia
-            ixx="4.78483605712844E-05"
-            ixy="1.42081909356751E-07"
-            ixz="8.32917079044309E-06"
-            iyy="5.42362047732042E-05"
-            iyz="-2.90608446019989E-08"
-            izz="3.36120409842199E-05" />
-      </inertial>
-      <visual>
-        <origin
-            xyz="0 0 0"
-            rpy="0 0 0" />
-        <geometry>
-          <mesh filename="package://${MESH_LINK_4_1}" />
-        </geometry>
-      </visual>
-      <collision>
-        <origin
-            xyz="0 0 0"
-            rpy="0 0 0" />
-        <geometry>
-          <mesh filename="package://${MESH_LINK_4_1}" />
-        </geometry>
+        <inertia ixx="4.78483605712844E-05" ixy="1.42081909356751E-07" ixz="8.32917079044309E-06"
+                 iyy="5.42362047732042E-05" iyz="-2.90608446019989E-08" izz="3.36120409842199E-05" />
+      </inertial>
+      <visual>
+        <origin xyz="0 0 0" rpy="0 0 0" />
+        <geometry><mesh filename="package://${MESH_LINK_4_1}" /></geometry>
+      </visual>
+      <collision>
+        <origin xyz="0 0 0" rpy="0 0 0" />
+        <geometry><mesh filename="package://${MESH_LINK_4_1}" /></geometry>
       </collision>
     </link>
     <link name="${prefix}mg400_link4_2">
       <inertial>
-        <origin
-            xyz="0.0876391591012518 0.023499867452275 0.00831492252441945"
-            rpy="0 0 0" />
+        <origin xyz="0.0876391591012518 0.023499867452275 0.00831492252441945" rpy="0 0 0" />
         <mass value="0.0453569016333092" />
-        <inertia
-            ixx="2.00037596001325E-05"
-            ixy="3.34474706250153E-09"
-            ixz="2.17594982354756E-07"
-            iyy="0.000132049841023893"
-            iyz="5.36978669669685E-10"
-            izz="0.000141813978894428" />
-      </inertial>
-      <visual>
-        <origin
-            xyz="0 0 0"
-            rpy="0 0 0" />
-        <geometry>
-          <mesh filename="package://${MESH_LINK_4_2}" />
-        </geometry>
-      </visual>
-      <collision>
-        <origin
-            xyz="0 0 0"
-            rpy="0 0 0" />
-        <geometry>
-          <mesh filename="package://${MESH_LINK_4_2}" />
-        </geometry>
+        <inertia ixx="2.00037596001325E-05" ixy="3.34474706250153E-09" ixz="2.17594982354756E-07"
+                 iyy="0.000132049841023893" iyz="5.36978669669685E-10" izz="0.000141813978894428" />
+      </inertial>
+      <visual>
+        <origin xyz="0 0 0" rpy="0 0 0" />
+        <geometry><mesh filename="package://${MESH_LINK_4_2}" /></geometry>
+      </visual>
+      <collision>
+        <origin xyz="0 0 0" rpy="0 0 0" />
+        <geometry><mesh filename="package://${MESH_LINK_4_2}" /></geometry>
       </collision>
     </link>
     <link name="${prefix}mg400_link4_3">
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