Commit message: Before direct trajectory refactor: stable build with bridge loop

File: src/MG400_ROS2/mg400_description/urdf/mg400.urdf.xacro (robot description, xacro)
@@ -42,13 +42,52 @@
     <gazebo reference="mg400_link5"><gravity>0</gravity></gazebo>
     <gazebo reference="mg400_end_effector_flange"><gravity>0</gravity></gazebo>
-   <gazebo>
-    <static>true</static>
-   </gazebo>
-   <gazebo>
-       <plugin name="gazebo_ros_joint_pose_trajectory" filename="libgazebo_ros_joint_pose_trajectory.so">
-           <ros>
-           </ros>
-           <update_rate>30</update_rate>
-       </plugin>
-   </gazebo>
+    <ros2_control name="GazeboSystem" type="system">
+        <hardware>
+            <plugin>gazebo_ros2_control/GazeboSystem</plugin>
+        </hardware>
+        <joint name="mg400_j1">
+            <command_interface name="position"/>  <state_interface name="position"/>
+            <state_interface name="velocity"/>
+        </joint>
+        <joint name="mg400_j2_1">
+            <command_interface name="position"/>
+            <state_interface name="position"/>
+            <state_interface name="velocity"/>
+        </joint>
+        <joint name="mg400_j2_2">
+            <command_interface name="position"/>
+            <state_interface name="position"/>
+            <state_interface name="velocity"/>
+        </joint>
+        <joint name="mg400_j3_1">
+            <command_interface name="position"/>
+            <state_interface name="position"/>
+            <state_interface name="velocity"/>
+        </joint>
+        <joint name="mg400_j3_2">
+            <command_interface name="position"/>
+            <state_interface name="position"/>
+            <state_interface name="velocity"/>
+        </joint>
+        <joint name="mg400_j4_1">
+            <command_interface name="position"/>
+            <state_interface name="position"/>
+            <state_interface name="velocity"/>
+        </joint>
+        <joint name="mg400_j4_2">
+            <command_interface name="position"/>
+            <state_interface name="position"/>
+            <state_interface name="velocity"/>
+        </joint>
+        <joint name="mg400_j5">
+            <command_interface name="position"/>
+            <state_interface name="position"/>
+            <state_interface name="velocity"/>
+        </joint>
+    </ros2_control>
+    <gazebo>
+        <plugin filename="libgazebo_ros2_control.so" name="gazebo_ros2_control">
+            <parameters>$(find dobot_gazebo)/config/controllers.yaml</parameters>
+        </plugin>
+    </gazebo>
 </robot>

File: src/MG400_ROS2/mg400_description/urdf/mg400.xacro (robot description, xacro)
@@ -233,6 +233,6 @@
       <child link="${prefix}mg400_link1" />
       <axis xyz="0 0 1" />
-      <limit lower="${-180.0 * const.TO_RADIAN}" upper="${180.0 * const.TO_RADIAN}" effort="0" velocity="0" />
-      <dynamics damping="100.0" friction="100.0"/>
+      <limit lower="${-180.0 * const.TO_RADIAN}" upper="${180.0 * const.TO_RADIAN}" effort="10000.0" velocity="5.0" />
+      <dynamics damping="50.0" friction="1.0"/>
     </joint>
     <joint name="${prefix}mg400_j2_1" type="revolute">
@@ -241,6 +241,6 @@
       <child link="${prefix}mg400_link2_1" />
       <axis xyz="0 1 0" />
-      <limit lower="-3.14" upper="3.14" effort="0" velocity="0" />
-      <dynamics damping="100.0" friction="100.0"/>
+      <limit lower="-3.14" upper="3.14" effort="10000.0" velocity="5.0" />
+      <dynamics damping="50.0" friction="1.0"/>
     </joint>
     <joint name="${prefix}mg400_j2_2" type="revolute">
@@ -249,6 +249,6 @@
       <child link="${prefix}mg400_link2_2" />
       <axis xyz="0 1 0" />
-      <limit lower="-3.14" upper="3.14" effort="0" velocity="0" />
-      <dynamics damping="100.0" friction="100.0"/>
+      <limit lower="-3.14" upper="3.14" effort="10000.0" velocity="5.0" />
+      <dynamics damping="50.0" friction="1.0"/>
     </joint>
     <joint name="${prefix}mg400_j3_1" type="revolute">
@@ -257,6 +257,6 @@
       <child link="${prefix}mg400_link3_1" />
       <axis xyz="0 1 0" />
-      <limit lower="-3.14" upper="3.14" effort="0" velocity="0" />
-      <dynamics damping="100.0" friction="100.0"/>
+      <limit lower="-3.14" upper="3.14" effort="10000.0" velocity="5.0" />
+      <dynamics damping="50.0" friction="1.0"/>
     </joint>
     <joint name="${prefix}mg400_j3_2" type="revolute">
@@ -265,6 +265,6 @@
       <child link="${prefix}mg400_link3_2" />
       <axis xyz="0 1 0" />
-      <limit lower="-3.14" upper="3.14" effort="0" velocity="0" />
-      <dynamics damping="100.0" friction="100.0"/>
+      <limit lower="-3.14" upper="3.14" effort="10000.0" velocity="5.0" />
+      <dynamics damping="50.0" friction="1.0"/>
     </joint>
     <joint name="${prefix}mg400_j4_1" type="revolute">
@@ -273,6 +273,6 @@
       <child link="${prefix}mg400_link4_1" />
       <axis xyz="0 1 0" />
-      <limit lower="-3.14" upper="3.14" effort="0" velocity="0" />
-      <dynamics damping="100.0" friction="100.0"/>
+      <limit lower="-3.14" upper="3.14" effort="10000.0" velocity="5.0" />
+      <dynamics damping="50.0" friction="1.0"/>
     </joint>
     <joint name="${prefix}mg400_j4_2" type="revolute">
@@ -281,6 +281,6 @@
       <child link="${prefix}mg400_link4_2" />
       <axis xyz="0 1 0" />
-      <limit lower="-3.14" upper="3.14" effort="0" velocity="0" />
-      <dynamics damping="100.0" friction="100.0"/>
+      <limit lower="-3.14" upper="3.14" effort="10000.0" velocity="5.0" />
+      <dynamics damping="50.0" friction="1.0"/>
     </joint>
     <joint name="${prefix}mg400_j4_3" type="fixed">
@@ -299,6 +299,6 @@
       <child link="${prefix}mg400_end_effector_flange" />
       <axis xyz="0 0 1" />
-      <limit lower="${-180.0 * const.TO_RADIAN}" upper="${180.0 * const.TO_RADIAN}" effort="0" velocity="0" />
-      <dynamics damping="100.0" friction="100.0"/>
+      <limit lower="${-180.0 * const.TO_RADIAN}" upper="${180.0 * const.TO_RADIAN}" effort="10000.0" velocity="5.0" />
+      <dynamics damping="50.0" friction="1.0"/>
     </joint>
   </xacro:macro>

Commit message: fix: стабільна фізика Gazebo, оптимізація колізій та робоча логіка IK

File: src/MG400_ROS2/mg400_description/urdf/mg400.urdf.xacro (robot description, xacro)
@@ -55,15 +55,5 @@
             <state_interface name="velocity"/>
         </joint>
-        <joint name="mg400_j2_2">
-            <command_interface name="position"/>
-            <state_interface name="position"/>
-            <state_interface name="velocity"/>
-        </joint>
         <joint name="mg400_j3_1">
-            <command_interface name="position"/>
-            <state_interface name="position"/>
-            <state_interface name="velocity"/>
-        </joint>
-        <joint name="mg400_j3_2">
             <command_interface name="position"/>
             <state_interface name="position"/>
@@ -75,10 +65,26 @@
             <state_interface name="velocity"/>
         </joint>
-        <joint name="mg400_j4_2">
+        <joint name="mg400_j5">
             <command_interface name="position"/>
             <state_interface name="position"/>
             <state_interface name="velocity"/>
         </joint>
-        <joint name="mg400_j5">
+        <joint name="mg400_j2_2">
+            <param name="mimic">mg400_j2_1</param>
+            <param name="multiplier">1</param>
+            <command_interface name="position"/>
+            <state_interface name="position"/>
+            <state_interface name="velocity"/>
+        </joint>
+        <joint name="mg400_j3_2">
+            <param name="mimic">mg400_j3_1</param>
+            <param name="multiplier">1</param>
+            <command_interface name="position"/>
+            <state_interface name="position"/>
+            <state_interface name="velocity"/>
+        </joint>
+        <joint name="mg400_j4_2">
+            <param name="mimic">mg400_j4_1</param>
+            <param name="multiplier">1</param>
             <command_interface name="position"/>
             <state_interface name="position"/>

File: src/MG400_ROS2/mg400_description/urdf/mg400.xacro (robot description, xacro)
@@ -1,9 +1,7 @@
 <?xml version="1.0" encoding="UTF-8"?>
 <robot xmlns:xacro="http://ros.org/wiki/xacro">
-  <!-- constants -->
   <xacro:include
       filename="$(find mg400_description)/urdf/common/constants.xacro"
       ns="const" />
-  <!-- Base path for meshes -->
   <xacro:property name="BASE_PATH" value="mg400_description/meshes" />
   <xacro:property name="MESH_BASE_LINK" value="${BASE_PATH}/base_link.dae" />
@@ -23,5 +21,4 @@
       <color rgba="0.2 0.0 0.0 0.5" />
     </material>
-    <!-- links -->
     <link name="${prefix}mg400_base_link">
       <inertial>
@@ -61,5 +58,5 @@
         <origin xyz="-0.00321788524756698 0.0352926570826593 0.0596131328734945" rpy="0 0 0" />
         <mass value="0.0866115884541459" />
-        <inertia ixx="0.000338551627157209" ixy="-2.78858228577314E-09" ixz="1.05212346076681E-05"
+        <inertia ixx="0.000338551627157209" ixy="-2.78858228577314E-09" ixz="0.15212346076681E-05"
                  iyy="0.000307789653713489" iyz="-1.36109590152488E-06" izz="3.89949940178023E-05" />
       </inertial>
@@ -158,5 +155,5 @@
         <mass value="0.01907" />
         <inertia ixx="3.28164E-05" ixy="3.15E-10" ixz="2.42378E-06"
-                 iyy="3.17191E-05" iyz="-1.27E-10" izz="1.08143E-05" />
+                 iyy="3.17191E-05" iyz="-1.27E-10" izz="0.18143E-05" />
       </inertial>
       <visual>
@@ -210,5 +207,4 @@
       </link>
     </xacro:if>
-    <!-- joints -->
     <joint name="${prefix}mg400_base_joint" type="fixed">
       <parent link="${parent}" />
@@ -234,5 +230,5 @@
       <axis xyz="0 0 1" />
       <limit lower="${-180.0 * const.TO_RADIAN}" upper="${180.0 * const.TO_RADIAN}" effort="10000.0" velocity="5.0" />
-      <dynamics damping="50.0" friction="1.0"/>
+      <dynamics damping="0.5" friction="0.1"/>
     </joint>
     <joint name="${prefix}mg400_j2_1" type="revolute">
@@ -242,5 +238,5 @@
       <axis xyz="0 1 0" />
       <limit lower="-3.14" upper="3.14" effort="10000.0" velocity="5.0" />
-      <dynamics damping="50.0" friction="1.0"/>
+      <dynamics damping="0.5" friction="0.1"/>
     </joint>
     <joint name="${prefix}mg400_j2_2" type="revolute">
@@ -250,5 +246,6 @@
       <axis xyz="0 1 0" />
       <limit lower="-3.14" upper="3.14" effort="10000.0" velocity="5.0" />
-      <dynamics damping="50.0" friction="1.0"/>
+      <dynamics damping="0.5" friction="0.1"/>
+      <mimic joint="${prefix}mg400_j2_1" multiplier="1" offset="0"/>
     </joint>
     <joint name="${prefix}mg400_j3_1" type="revolute">
@@ -258,5 +255,5 @@
       <axis xyz="0 1 0" />
       <limit lower="-3.14" upper="3.14" effort="10000.0" velocity="5.0" />
-      <dynamics damping="50.0" friction="1.0"/>
+      <dynamics damping="0.5" friction="0.1"/>
     </joint>
     <joint name="${prefix}mg400_j3_2" type="revolute">
@@ -266,5 +263,6 @@
       <axis xyz="0 1 0" />
       <limit lower="-3.14" upper="3.14" effort="10000.0" velocity="5.0" />
-      <dynamics damping="50.0" friction="1.0"/>
+      <dynamics damping="0.5" friction="0.1"/>
+      <mimic joint="${prefix}mg400_j3_1" multiplier="1" offset="0"/>
     </joint>
     <joint name="${prefix}mg400_j4_1" type="revolute">
@@ -274,5 +272,5 @@
       <axis xyz="0 1 0" />
       <limit lower="-3.14" upper="3.14" effort="10000.0" velocity="5.0" />
-      <dynamics damping="50.0" friction="1.0"/>
+      <dynamics damping="0.5" friction="0.1"/>
     </joint>
     <joint name="${prefix}mg400_j4_2" type="revolute">
@@ -282,5 +280,6 @@
       <axis xyz="0 1 0" />
       <limit lower="-3.14" upper="3.14" effort="10000.0" velocity="5.0" />
-      <dynamics damping="50.0" friction="1.0"/>
+      <dynamics damping="0.5" friction="0.1"/>
+      <mimic joint="${prefix}mg400_j4_1" multiplier="1" offset="0"/>
     </joint>
     <joint name="${prefix}mg400_j4_3" type="fixed">
@@ -300,5 +299,5 @@
       <axis xyz="0 0 1" />
       <limit lower="${-180.0 * const.TO_RADIAN}" upper="${180.0 * const.TO_RADIAN}" effort="10000.0" velocity="5.0" />
-      <dynamics damping="50.0" friction="1.0"/>
+      <dynamics damping="0.5" friction="0.1"/>
     </joint>
   </xacro:macro>
